File: avocado/avocado_v1.0.sch (EAGLE design)
At the start: 106 parts, among them IC1 TM4C129XXXPDT, IC3 MAX31855, IC4 ISO3088, J1 1X2-3.5MM, U1 LMT87DCKT, U2 AS5048A-HTSP-500

Commit message: finished adding parts for motor
Parts:
- removed USR_SW1, USR_SW2: B3S-10XX, avocado:B3S-10XX
- added C38, C39, C40: 2200pF, rcl:C-USC0805
- added C41, C42, C43: 1000pF, rcl:C-USC0805
- added R12: 120, rcl:R-US_R0805
- added R15, R26, R36, R38: 7.5K, rcl:R-US_R0805
- added R16, R17, R35, R37: 84.5K, rcl:R-US_R0805
- added U$13, U$8: UPJXXXXXMHD6, avocado:UPJXXXXXMHD6
- added U$6: MHSS1105, avocado:MHSS1105
- added U$7: TPD4S009, avocado:TPD4S009
- added ZERO: B3F-60XX, avocado:B3F-60XX
- C14, C15, C34: value 10nF -> 4.7nF
- RESET, WAKE: value B3S-10XX -> B3F-60XX; device avocado:B3S-10XX -> avocado:B3F-60XX
Connections:
- removed net N$5 (its old number): C5.1, C6.1, C7.1, U$10.VIN, U$11.VIN, U$12.VIN, U$9.VDRAIN
- new net N$18: R12.2, U$6.2
- new net VSENS1: R15.2, R16.1, U$7.D1+
- new net VSENS2: R17.1, R26.2, U$7.D2+
- new net VSENS3: R35.1, R36.2, U$7.D2-
- new net VSENSVM: R37.1, R38.2, U$7.D1-
- net 24VDC: now also C5.1, C6.1, C7.1, R37.2, U$10.VIN, U$11.VIN, U$12.VIN, U$13.A, U$8.A, U$9.VDRAIN
- net 3V3DC: now also U$7.VCC
- net A: now also U$6.COM
- net B: now also R12.1
- net GND: now also C38.2, C39.2, C40.2, C41.2, C42.2, C43.2, R15.1, R26.1, R36.1, R38.1, RESET.2, U$13.C, U$7.GND, U$8.C, WAKE.2, ZERO.2; no longer RESET.S, RESET.S1, USR_SW1.S, USR_SW1.S1, USR_SW2.S, USR_SW2.S1, WAKE.S, WAKE.S1
- net H1: now also C42.1
- net H2: now also C41.1
- net H3: now also C43.1
- net M1: now also R16.2
- net M2: now also R17.2
- net M3: now also R35.2
- net NTRST: now also RESET.1; no longer RESET.P, RESET.P1
- net NWAKE: now also WAKE.1; no longer WAKE.P, WAKE.P1
- net PD5: now also C40.1
- net PD6: now also C39.1
- net PD7: now also C38.1
- net PJ0: now also ZERO.1; no longer USR_SW1.P, USR_SW1.P1
- net PJ1: no longer USR_SW2.P, USR_SW2.P1
Other:
- moved on the sheet: C12, C14, C15, C19, C33, C34, C35, C37, C5, C6, C7, D2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

Commit message: started board layout
Parts:
- removed C26, C36: 0.1uF, rcl:C-USC0805
- removed C31, C32: 1uF, rcl:C-USC0805
- removed J4: (no value), SparkFun-Connectors:CONN_07
- removed R12: 120, rcl:R-US_R0805
- removed RESET, WAKE, ZERO: B3F-60XX, avocado:B3F-60XX
- removed U$6: MHSS1105, avocado:MHSS1105
- removed U2: AS5048A-HTSP-500, avocado:AS5048A-HTSP-500
- C11, C12, C13, C16, C17, C18, C19, C20, C21, C22, C23, C24, C25, C27, C28, C29, C30, C33, C35, C37, C38, C39, C40, C41, C42, C43, C8: device rcl:C-USC0805 -> rcl:C-USC0402
- J2: device avocado:61200621621 -> SparkFun-Connectors:CONN_04
- J3: device avocado:61200621621 -> SparkFun-Connectors:CONN_04X2
- R1: value 100 -> 330; device rcl:R-US_R0805 -> rcl:R-US_R0402
- R13, R14, R15, R16, R17, R18, R19, R20, R21, R22, R23, R24, R25, R26, R27, R28, R29, R30, R31, R32, R35, R36, R37, R38, R7, R8: device rcl:R-US_R0805 -> rcl:R-US_R0402
- R2, R3: device SparkFun-Resistors:0.3OHM-0805-1/8W-1% -> rcl:R-US_R0402
- R33, R34: device adafruit:R-US_R0805 -> adafruit:R-US_R0402
- U$1, U$2: value S03B-PASK-2 -> 0522070633; device avocado:S03B-PASK-2 -> avocado:0522070633
- U$5: value B2PS-VH -> 5040500691; device avocado:B2PS-VH -> avocado:5040500691
- U$9: value DRV8323S_AVOCADODRV8323S_AVOCADO -> DRV8323SHOMEMADE; device motor_control:DRV8323S_AVOCADODRV8323S_AVOCADO -> motor_control:DRV8323SHOMEMADE
Connections:
- net N$10 renamed GL1
- net N$11 renamed DVDD
- net N$26 renamed ISENS2
- net N$29 renamed GH1
- net N$30 renamed SH1
- net N$32 renamed GH2
- net N$33 renamed SH2
- net N$34 renamed GL2
- net N$35 renamed GH3
- net N$36 renamed SH3
- net N$37 renamed GL3
- net N$38 renamed ISENS3
- net N$49 renamed NFAULT
- net N$5 renamed ISENS1
- removed net ENC_CLK: J2.2, U2.CLK
- removed net ENC_GND: J2.6
- removed net ENC_MISO: U2.MISO
- removed net ENC_MOSI: J2.3, U2.MOSI
- removed net ENC_PWR: C31.1, C32.1, J2.4, U2.VDD3V, U2.VDD5V
- removed net ENC_SS: J2.1, U2.!CSN
- removed net N$18: R12.2, U$6.2
- removed net N$20: D6.A, R3.2
- removed net N$51: J2.5
- new net N$7: D6.A, R2.2
- net 24VDC: now also J2.1, J2.2; no longer IC4.VCC2, U$5.PWR
- net 3V3DC: now also R2.1, U$1.P$2, U$2.P$2; no longer C26.1, C36.1, J3.4, R3.1
- net 5VDC: now also IC4.VCC2, R3.1; no longer R2.1
- net A: now also U$1.P$6; no longer U$1.P$1, U$2.P$1, U$6.COM
- net B: now also U$1.P$5; no longer R12.1, U$1.P$2, U$2.P$2
- net GND: now also J2.3, J2.4, U$1.P$3, U$2.P$1, U$5.2, U$5.4, U$5.6; no longer C26.2, C31.2, C32.2, C36.2, J3.6, RESET.2, U$5.GND, U2.GND, WAKE.2, ZERO.2
- net GND_EXT: now also U$1.P$4; no longer U$1.P$3, U$2.P$3
- net N$19: now also R3.2; no longer R2.2
- net NTRST: now also J3.7, U$5.1; no longer J4.7, RESET.1
- net NWAKE: now also U$5.3; no longer WAKE.1
- net PA0: now also J3.2; no longer J4.2
- net PA1: now also J3.1; no longer J4.1
- net PA2: now also U$2.P$5; no longer J3.2
- net PA3: now also U$2.P$6; no longer J3.1
- net PA4: now also U$2.P$4; no longer J3.3
- net PA5: now also U$2.P$3; no longer J3.5
- net PJ0: now also U$5.5; no longer ZERO.1
- net SWCLK: now also J3.3; no longer J4.3
- net SWDIO: now also J3.4; no longer J4.4
- net SWO: now also J3.6; no longer J4.6
- net TDI: now also J3.5; no longer J4.5
Other:
- moved on the sheet: 3V3BUCK, 5VBUCK, C1, C2, C27, C3, C4, D1, D4, D6, D7, IC4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

Commit message: made significant routing progress
Connections:
- removed net PC7: IC1.PC6, IC1.PC7
- removed net PE5: IC1.PE5
- removed net PK0: IC1.PK0
- removed net PK1: IC1.PK1
- removed net PK2: IC1.PK2
- net PA6: now also U$5.5
- net PC6: now also IC1.PC6, IC1.PC7
- net PD5: now also C38.1, U$9.SOA; no longer C40.1, U$9.SOC
- net PD7: now also C40.1, U$9.SOC; no longer C38.1, U$9.SOA
- net PF3: no longer U$9.INLC
- net PF4: no longer U$9.INHC
- net PJ0: no longer U$5.5
- net PP0: now also U$9.INLC
- net PP1: now also U$9.INHC
- net VSENS1: now also IC1.PK0
- net VSENS2: now also IC1.PK1
- net VSENS3: now also IC1.PK2
- net VSENSVM: now also IC1.PE5
