File: avocado/avocado_v2.0.sch (EAGLE design)
At the start: 99 parts, among them IC1 TM4C129XXXPDT, IC3 MAX31855, IC4 ISO3088, J1 THERMOCOUPLE, U1 LMT87DCKT

Commit message: added v2.0 of the avocado main pcb
Parts:
- removed D7: BLUE, SparkFun-LED:LED-BLUE0603
- removed J2: (no value), SparkFun-Connectors:CONN_04
- removed OPTBIT0, OPTBIT1, OPTBIT2, OPTBIT3: (no value), avocado:QRE1113
- removed R19, R27, R29, R31: 100, rcl:R-US_R0402
- removed R20, R28, R30, R32: 10K, rcl:R-US_R0402
- removed R3: 330, rcl:R-US_R0402
- added C31, C32: 1uF, rcl:C-USC0805
- added C52, C53, C54, C55, C56: C7563, avocado:C7563
- added R16: 120, rcl:R-US_R0805
- added U$17: MHSS1105, avocado:MHSS1105
- added U2: AS5048A-HTSP-500, avocado:AS5048A-HTSP-500
- U$2: value 0522070633 -> 5040500691; device avocado:0522070633 -> avocado:5040500691
- U$5: value 5040500591 -> S03B-PASK-2; device avocado:5040500591 -> avocado:S03B-PASK-2
Connections:
- removed net N$12: OPTBIT1.A, R29.1
- removed net N$14: OPTBIT0.A, R31.1
- removed net N$19: D7.A, R3.2
- removed net N$4: OPTBIT3.A, R19.1
- removed net N$9: OPTBIT2.A, R27.1
- new net N$23: R16.2, U$17.2
- net 24VDC: now also C52.1, C53.1, C54.1, C55.1, C56.1; no longer J2.1, J2.2
- net 3V3DC: now also C31.1, C32.1, U$2.2, U2.VDD3V, U2.VDD5V; no longer R19.2, R20.2, R27.2, R28.2, R29.2, R30.2, R31.2, R32.2, U$2.P$2, U$5.1
- net 5VDC: no longer R3.1
- net A: now also U$17.COM, U$5.P$1; no longer U$5.4
- net B: now also R16.1, U$5.P$2; no longer U$5.5
- net GND: now also C31.2, C32.2, C52.2, C53.2, C54.2, C55.2, C56.2, U$2.1, U2.GND; no longer D7.C, J2.3, J2.4, OPTBIT0.E, OPTBIT0.K, OPTBIT1.E, OPTBIT1.K, OPTBIT2.E, OPTBIT2.K, OPTBIT3.E, OPTBIT3.K, U$2.P$1, U$5.2
- net GND_EXT: now also U$5.P$3; no longer U$5.3
- net PA2: now also U2.CLK; no longer U$2.P$5
- net PA3: now also U2.!CSN; no longer U$2.P$6
- net PA4: now also U2.MOSI; no longer U$2.P$4
- net PA5: now also U2.MISO; no longer U$2.P$3
- net PE0: now also U$2.6; no longer OPTBIT0.C, R32.1
- net PE1: now also U$2.5; no longer OPTBIT1.C, R30.1
- net PE2: now also U$2.4; no longer OPTBIT2.C, R28.1
- net PE3: now also U$2.3; no longer OPTBIT3.C, R20.1
- net PE4: no longer IC3.DO
- net PE5: now also IC3.DO
Other:
- moved on the sheet: IC4, U$2

Commit message: version 2 of the avocado pcb finished
Parts:
- removed U$6: LM2594M-5.0, avocado:LM2594M-5.0
- added C16: 0.01uF, rcl:C-USC0402
- added U$8: LM2675M, avocado:LM2675M
- L2: value SRU1028 -> B82464G4473M000; device avocado:SRU1028 -> avocado:B82464G4473M000
Connections:
- new net N$4: C16.1, U$8.CB
- net 24VDC: now also U$8.VIN; no longer U$6.VIN
- net 3V3DC: now also U$8.FB; no longer U$6.FB
- net GND: now also J3.8, U$8.GND; no longer U$6.GND, U$6.ON/OFF
- net N$25: now also C16.2, U$8.VSW; no longer U$6.OUT
Other:
- moved on the sheet: C3, C4, D4, D6, L2, R2
Changed lines of the file:
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@@
 <part name="FB2" library="microbuilder" deviceset="FERRITE" device="_0805" value="Ferrite"/>
 <part name="U$7" library="avocado" deviceset="LM2594M-5.0" device=""/>
-<part name="U$6" library="avocado" deviceset="LM2594M-5.0" device=""/>
 <part name="D1" library="avocado" deviceset="MBRS130LT3" device=""/>
 <part name="D4" library="avocado" deviceset="MBRS130LT3" device=""/>
@@
 <part name="C4" library="avocado" deviceset="AVX_TPS_CAP" device="D" value="15u"/>
 <part name="L1" library="avocado" deviceset="SRU1028" device=""/>
-<part name="L2" library="avocado" deviceset="SRU1028" device=""/>
 <part name="GND1" library="SparkFun-PowerSymbols" deviceset="GND" device=""/>
 <part name="GND2" library="SparkFun-PowerSymbols" deviceset="GND" device=""/>
@@
 <part name="C32" library="rcl" library_urn="urn:adsk.eagle:library:334" deviceset="C-US" device="C0805" package3d_urn="urn:adsk.eagle:package:23617/2" value="1uF"/>
 <part name="U$2" library="avocado" deviceset="5040500691" device=""/>
+<part name="C16" library="rcl" library_urn="urn:adsk.eagle:library:334" deviceset="C-US" device="C0402" package3d_urn="urn:adsk.eagle:package:23626/1" value="0.01uF"/>
+<part name="U$8" library="avocado" deviceset="LM2675" device="M"/>
+<part name="L2" library="avocado" deviceset="B82464G4473M000" device=""/>
 </parts>
 <sheets>
@@
 <instance part="FB2" gate="G$1" x="157.48" y="-106.68"/>
 <instance part="U$7" gate="A" x="-233.68" y="129.54"/>
-<instance part="U$6" gate="A" x="-231.14" y="63.5"/>
 <instance part="D1" gate="G$1" x="-213.36" y="127" rot="R90"/>
-<instance part="D4" gate="G$1" x="-213.36" y="60.96" rot="R90"/>
+<instance part="D4" gate="G$1" x="-213.36" y="50.8" rot="R90"/>
 <instance part="C1" gate="G$1" x="-195.58" y="129.54"/>
 <instance part="C2" gate="G$1" x="-261.62" y="132.08"/>
-<instance part="C3" gate="G$1" x="-198.12" y="63.5"/>
-<instance part="C4" gate="G$1" x="-259.08" y="63.5"/>
+<instance part="C3" gate="G$1" x="-198.12" y="53.34"/>
+<instance part="C4" gate="G$1" x="-259.08" y="66.04"/>
 <instance part="L1" gate="G$1" x="-203.2" y="137.16" smashed="yes" rot="R90">
 <attribute name="NAME" x="-205.74" y="138.43" size="1.778" layer="95" font="vector" rot="R90"/>
 <attribute name="VALUE" x="-200.66" y="138.43" size="1.778" layer="96" font="vector" rot="R90" align="top-left"/>
 </instance>
-<instance part="L2" gate="G$1" x="-205.74" y="71.12" smashed="yes" rot="R90">
-<attribute name="NAME" x="-208.28" y="72.39" size="1.778" layer="95" font="vector" rot="R90"/>
-<attribute name="VALUE" x="-203.2" y="72.39" size="1.778" layer="96" font="vector" rot="R90" align="top-left"/>
-</instance>
 <instance part="GND1" gate="1" x="-205.74" y="111.76"/>
 <instance part="GND2" gate="1" x="-254" y="111.76"/>
-<instance part="GND8" gate="1" x="-254" y="45.72"/>
-<instance part="GND29" gate="1" x="-205.74" y="45.72"/>
+<instance part="GND8" gate="1" x="-259.08" y="50.8"/>
+<instance part="GND29" gate="1" x="-205.74" y="35.56"/>
 <instance part="IC4" gate="G$1" x="-241.3" y="-7.62"/>
 <instance part="U$9" gate="G$1" x="-17.78" y="-106.68"/>
@@
 <instance part="GND9" gate="1" x="-76.2" y="-76.2"/>
 <instance part="GND48" gate="1" x="-91.44" y="-76.2"/>
-<instance part="R2" gate="G$1" x="-187.96" y="63.5" smashed="yes" rot="R270">
-<attribute name="NAME" x="-186.4614" y="67.31" size="1.778" layer="95" rot="R270"/>
-<attribute name="VALUE" x="-191.262" y="67.31" size="1.778" layer="96" rot="R270"/>
+<instance part="R2" gate="G$1" x="-187.96" y="53.34" smashed="yes" rot="R270">
+<attribute name="NAME" x="-186.4614" y="57.15" size="1.778" layer="95" rot="R270"/>
+<attribute name="VALUE" x="-191.262" y="57.15" size="1.778" layer="96" rot="R270"/>
 </instance>
-<instance part="D6" gate="G$1" x="-187.96" y="55.88"/>
-<instance part="GND49" gate="1" x="-187.96" y="45.72"/>
+<instance part="D6" gate="G$1" x="-187.96" y="45.72"/>
+<instance part="GND49" gate="1" x="-187.96" y="35.56"/>
 <instance part="J3" gate="G$1" x="149.86" y="78.74"/>
 <instance part="R12" gate="G$1" x="78.74" y="35.56" smashed="yes" rot="R180">
@@
 <instance part="C32" gate="G$1" x="-175.26" y="-78.74"/>
 <instance part="U$2" gate="G$1" x="-195.58" y="-147.32"/>
+<instance part="C16" gate="G$1" x="-218.44" y="66.04" rot="R90"/>
+<instance part="U$8" gate="A" x="-233.68" y="66.04"/>
+<instance part="L2" gate="G$1" x="-205.74" y="60.96" rot="R90"/>
 </instances>
 <busses>
@@
 </segment>
 <segment>
-<pinref part="U$6" gate="A" pin="VIN"/>
-<wire x1="-248.92" y1="71.12" x2="-259.08" y2="71.12" width="0.1524" layer="91"/>
+<wire x1="-243.84" y1="71.12" x2="-259.08" y2="71.12" width="0.1524" layer="91"/>
 <pinref part="C4" gate="G$1" pin="A"/>
-<wire x1="-259.08" y1="71.12" x2="-259.08" y2="68.58" width="0.1524" layer="91"/>
 <label x="-259.08" y="71.12" size="1.778" layer="95"/>
+<pinref part="U$8" gate="A" pin="VIN"/>
 </segment>
 <segment>
@@
 <segment>
 <pinref part="C4" gate="G$1" pin="C"/>
-<wire x1="-259.08" y1="58.42" x2="-259.08" y2="48.26" width="0.1524" layer="91"/>
-<pinref part="U$6" gate="A" pin="GND"/>
-<wire x1="-259.08" y1="48.26" x2="-254" y2="48.26" width="0.1524" layer="91"/>
-<pinref part="U$6" gate="A" pin="ON/OFF"/>
-<wire x1="-254" y1="48.26" x2="-248.92" y2="48.26" width="0.1524" layer="91"/>
-<wire x1="-248.92" y1="63.5" x2="-254" y2="63.5" width="0.1524" layer="91"/>
-<wire x1="-254" y1="63.5" x2="-254" y2="48.26" width="0.1524" layer="91"/>
-<junction x="-254" y="48.26"/>
+<wire x1="-259.08" y1="60.96" x2="-259.08" y2="53.34" width="0.1524" layer="91"/>
 <pinref part="GND8" gate="1" pin="GND"/>
+<pinref part="U$8" gate="A" pin="GND"/>
+<wire x1="-243.84" y1="60.96" x2="-259.08" y2="60.96" width="0.1524" layer="91"/>
+<junction x="-259.08" y="60.96"/>
 </segment>
 <segment>
 <pinref part="C3" gate="G$1" pin="C"/>
-<wire x1="-198.12" y1="58.42" x2="-198.12" y2="48.26" width="0.1524" layer="91"/>
-<wire x1="-198.12" y1="48.26" x2="-205.74" y2="48.26" width="0.1524" layer="91"/>
+<wire x1="-198.12" y1="48.26" x2="-198.12" y2="38.1" width="0.1524" layer="91"/>
+<wire x1="-198.12" y1="38.1" x2="-205.74" y2="38.1" width="0.1524" layer="91"/>
 <pinref part="D4" gate="G$1" pin="A"/>
-<wire x1="-205.74" y1="48.26" x2="-213.36" y2="48.26" width="0.1524" layer="91"/>
-<wire x1="-213.36" y1="48.26" x2="-213.36" y2="58.42" width="0.1524" layer="91"/>
+<wire x1="-205.74" y1="38.1" x2="-213.36" y2="38.1" width="0.1524" layer="91"/>
+<wire x1="-213.36" y1="38.1" x2="-213.36" y2="48.26" width="0.1524" layer="91"/>
 <pinref part="GND29" gate="1" pin="GND"/>
-<junction x="-205.74" y="48.26"/>
+<junction x="-205.74" y="38.1"/>
 </segment>
 <segment>
@@
 <segment>
 <pinref part="D6" gate="G$1" pin="C"/>
-<wire x1="-187.96" y1="50.8" x2="-187.96" y2="48.26" width="0.1524" layer="91"/>
+<wire x1="-187.96" y1="40.64" x2="-187.96" y2="38.1" width="0.1524" layer="91"/>
 <pinref part="GND49" gate="1" pin="GND"/>
 </segment>
@@
 <wire x1="-190.5" y1="-139.7" x2="-177.8" y2="-139.7" width="0.1524" layer="91"/>
 <label x="-187.96" y="-139.7" size="1.778" layer="95"/>
+</segment>
+<segment>
+<pinref part="J3" gate="G$1" pin="8"/>
+<wire x1="157.48" y1="76.2" x2="167.64" y2="76.2" width="0.1524" layer="91"/>
+<label x="157.48" y="76.2" size="1.778" layer="95"/>
 </segment>
 </net>
@@
 </segment>
 <segment>
+<wire x1="-200.66" y1="60.96" x2="-198.12" y2="60.96" width="0.1524" layer="91"/>
+<pinref part="C3" gate="G$1" pin="A"/>
+<wire x1="-198.12" y1="60.96" x2="-198.12" y2="58.42" width="0.1524" layer="91"/>
+<wire x1="-198.12" y1="60.96" x2="-187.96" y2="60.96" width="0.1524" layer="91"/>
+<junction x="-198.12" y="60.96"/>
+<label x="-193.04" y="60.96" size="1.778" layer="95"/>
+<pinref part="R2" gate="G$1" pin="1"/>
+<wire x1="-187.96" y1="60.96" x2="-185.42" y2="60.96" width="0.1524" layer="91"/>
+<wire x1="-187.96" y1="60.96" x2="-187.96" y2="58.42" width="0.1524" layer="91"/>
+<junction x="-187.96" y="60.96"/>
+<pinref part="U$8" gate="A" pin="FB"/>
+<wire x1="-198.12" y1="60.96" x2="-198.12" y2="71.12" width="0.1524" layer="91"/>
+<wire x1="-198.12" y1="71.12" x2="-220.98" y2="71.12" width="0.1524" layer="91"/>
 <pinref part="L2" gate="G$1" pin="2"/>
-<wire x1="-200.66" y1="71.12" x2="-198.12" y2="71.12" width="0.1524" layer="91"/>
-<pinref part="C3" gate="G$1" pin="A"/>
-<wire x1="-198.12" y1="71.12" x2="-198.12" y2="68.58" width="0.1524" layer="91"/>
-<wire x1="-198.12" y1="71.12" x2="-187.96" y2="71.12" width="0.1524" layer="91"/>
-<junction x="-198.12" y="71.12"/>
-<label x="-193.04" y="71.12" size="1.778" layer="95"/>
-<pinref part="R2" gate="G$1" pin="1"/>
-<wire x1="-187.96" y1="71.12" x2="-185.42" y2="71.12" width="0.1524" layer="91"/>
-<wire x1="-187.96" y1="71.12" x2="-187.96" y2="68.58" width="0.1524" layer="91"/>
-<junction x="-187.96" y="71.12"/>
-</segment>
-<segment>
-<pinref part="U$6" gate="A" pin="FB"/>
-<wire x1="-248.92" y1="66.04" x2="-256.54" y2="66.04" width="0.1524" layer="91"/>
-<label x="-256.54" y="66.04" size="1.778" layer="95"/>
 </segment>
 <segment>
@@
 <net name="N$25" class="0">
 <segment>
-<pinref part="U$6" gate="A" pin="OUT"/>
 <pinref part="D4" gate="G$1" pin="C"/>
-<wire x1="-213.36" y1="71.12" x2="-213.36" y2="63.5" width="0.1524" layer="91"/>
+<wire x1="-213.36" y1="60.96" x2="-213.36" y2="53.34" width="0.1524" layer="91"/>
+<wire x1="-213.36" y1="60.96" x2="-210.82" y2="60.96" width="0.1524" layer="91"/>
+<pinref part="U$8" gate="A" pin="VSW"/>
+<wire x1="-220.98" y1="60.96" x2="-213.36" y2="60.96" width="0.1524" layer="91"/>
+<junction x="-213.36" y="60.96"/>
+<pinref part="C16" gate="G$1" pin="2"/>
+<wire x1="-213.36" y1="60.96" x2="-213.36" y2="66.04" width="0.1524" layer="91"/>
 <pinref part="L2" gate="G$1" pin="1"/>
-<wire x1="-213.36" y1="71.12" x2="-210.82" y2="71.12" width="0.1524" layer="91"/>
-<junction x="-213.36" y="71.12"/>
 </segment>
 </net>
@@
 </segment>
 </net>
+<net name="N$4" class="0">
+<segment>
+<pinref part="U$8" gate="A" pin="CB"/>
+<pinref part="C16" gate="G$1" pin="1"/>
+</segment>
+</net>

Commit message: latest gerbers and main pcb design
Parts:
- removed U2: AS5048A-HTSP-500, avocado:AS5048A-HTSP-500
- added U$1: 5040500691, avocado:5040500691
- U$2: value 5040500691 -> AS5048A-HTSP-500; device avocado:5040500691 -> avocado:AS5048A-HTSP-500
Connections:
- net 3V3DC: now also U$1.2, U$2.VDD3V, U$2.VDD5V; no longer U$2.2, U2.VDD3V, U2.VDD5V
- net GND: now also U$1.1, U$2.GND; no longer U$2.1, U2.GND
- net PA2: now also U$2.CLK; no longer U2.CLK
- net PA3: now also U$2.!CSN; no longer U2.!CSN
- net PA4: now also U$2.MOSI; no longer U2.MOSI
- net PA5: now also U$2.MISO; no longer U2.MISO
- net PE0: now also U$1.6; no longer U$2.6
- net PE1: now also U$1.5; no longer U$2.5
- net PE2: now also U$1.4; no longer U$2.4
- net PE3: now also U$1.3; no longer U$2.3
Changed lines of the file:
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@@
 <part name="U$17" library="avocado" deviceset="MHSS1105" device=""/>
 <part name="R16" library="rcl" library_urn="urn:adsk.eagle:library:334" deviceset="R-US_" device="R0805" package3d_urn="urn:adsk.eagle:package:23553/2" value="120"/>
-<part name="U2" library="avocado" deviceset="AS5048A-HTSP-500" device=""/>
+<part name="U$2" library="avocado" deviceset="AS5048A-HTSP-500" device=""/>
 <part name="C31" library="rcl" library_urn="urn:adsk.eagle:library:334" deviceset="C-US" device="C0805" package3d_urn="urn:adsk.eagle:package:23617/2" value="1uF"/>
 <part name="C32" library="rcl" library_urn="urn:adsk.eagle:library:334" deviceset="C-US" device="C0805" package3d_urn="urn:adsk.eagle:package:23617/2" value="1uF"/>
-<part name="U$2" library="avocado" deviceset="5040500691" device=""/>
+<part name="U$1" library="avocado" deviceset="5040500691" device=""/>
 <part name="C16" library="rcl" library_urn="urn:adsk.eagle:library:334" deviceset="C-US" device="C0402" package3d_urn="urn:adsk.eagle:package:23626/1" value="0.01uF"/>
 <part name="U$8" library="avocado" deviceset="LM2675" device="M"/>
@@
 <instance part="U$17" gate="G$1" x="-147.32" y="-10.16" rot="R270"/>
 <instance part="R16" gate="G$1" x="-134.62" y="-12.7" rot="R180"/>
-<instance part="U2" gate="G$1" x="-205.74" y="-88.9"/>
+<instance part="U$2" gate="G$1" x="-205.74" y="-88.9"/>
 <instance part="C31" gate="G$1" x="-182.88" y="-81.28"/>
 <instance part="C32" gate="G$1" x="-175.26" y="-78.74"/>
-<instance part="U$2" gate="G$1" x="-195.58" y="-147.32"/>
+<instance part="U$1" gate="G$1" x="-195.58" y="-147.32"/>
 <instance part="C16" gate="G$1" x="-218.44" y="66.04" rot="R90"/>
 <instance part="U$8" gate="A" x="-233.68" y="66.04"/>
@@
 </segment>
 <segment>
-<pinref part="U2" gate="G$1" pin="GND"/>
+<pinref part="U$2" gate="G$1" pin="GND"/>
 <wire x1="-190.5" y1="-104.14" x2="-182.88" y2="-104.14" width="0.1524" layer="91"/>
 <wire x1="-182.88" y1="-104.14" x2="-180.34" y2="-104.14" width="0.1524" layer="91"/>
@@
 </segment>
 <segment>
-<pinref part="U$2" gate="G$1" pin="1"/>
+<pinref part="U$1" gate="G$1" pin="1"/>
 <wire x1="-190.5" y1="-139.7" x2="-177.8" y2="-139.7" width="0.1524" layer="91"/>
 <label x="-187.96" y="-139.7" size="1.778" layer="95"/>
@@
 </segment>
 <segment>
-<pinref part="U2" gate="G$1" pin="VDD3V"/>
+<pinref part="U$2" gate="G$1" pin="VDD3V"/>
 <wire x1="-190.5" y1="-78.74" x2="-182.88" y2="-78.74" width="0.1524" layer="91"/>
 <label x="-190.5" y="-78.74" size="1.778" layer="95"/>
@@
 </segment>
 <segment>
-<pinref part="U2" gate="G$1" pin="VDD5V"/>
+<pinref part="U$2" gate="G$1" pin="VDD5V"/>
 <wire x1="-190.5" y1="-76.2" x2="-175.26" y2="-76.2" width="0.1524" layer="91"/>
 <label x="-187.96" y="-76.2" size="1.778" layer="95"/>
@@
 </segment>
 <segment>
-<pinref part="U$2" gate="G$1" pin="2"/>
+<pinref part="U$1" gate="G$1" pin="2"/>
 <wire x1="-190.5" y1="-142.24" x2="-177.8" y2="-142.24" width="0.1524" layer="91"/>
 <label x="-187.96" y="-142.24" size="1.778" layer="95"/>
@@
 </segment>
 <segment>
-<pinref part="U$2" gate="G$1" pin="3"/>
+<pinref part="U$1" gate="G$1" pin="3"/>
 <wire x1="-190.5" y1="-144.78" x2="-177.8" y2="-144.78" width="0.1524" layer="91"/>
 <label x="-187.96" y="-144.78" size="1.778" layer="95"/>
@@
 </segment>
 <segment>
-<pinref part="U$2" gate="G$1" pin="4"/>
+<pinref part="U$1" gate="G$1" pin="4"/>
 <wire x1="-190.5" y1="-147.32" x2="-177.8" y2="-147.32" width="0.1524" layer="91"/>
 <label x="-187.96" y="-147.32" size="1.778" layer="95"/>
@@
 </segment>
 <segment>
-<pinref part="U$2" gate="G$1" pin="5"/>
+<pinref part="U$1" gate="G$1" pin="5"/>
 <wire x1="-190.5" y1="-149.86" x2="-177.8" y2="-149.86" width="0.1524" layer="91"/>
 <label x="-187.96" y="-149.86" size="1.778" layer="95"/>
@@
 </segment>
 <segment>
-<pinref part="U$2" gate="G$1" pin="6"/>
+<pinref part="U$1" gate="G$1" pin="6"/>
 <wire x1="-190.5" y1="-152.4" x2="-177.8" y2="-152.4" width="0.1524" layer="91"/>
 <label x="-187.96" y="-152.4" size="1.778" layer="95"/>
@@
 </segment>
 <segment>
-<pinref part="U2" gate="G$1" pin="CLK"/>
+<pinref part="U$2" gate="G$1" pin="CLK"/>
 <wire x1="-220.98" y1="-78.74" x2="-231.14" y2="-78.74" width="0.1524" layer="91"/>
 <label x="-231.14" y="-78.74" size="1.778" layer="95"/>
@@
 </segment>
 <segment>
-<pinref part="U2" gate="G$1" pin="!CSN"/>
+<pinref part="U$2" gate="G$1" pin="!CSN"/>
 <wire x1="-220.98" y1="-76.2" x2="-231.14" y2="-76.2" width="0.1524" layer="91"/>
 <label x="-231.14" y="-76.2" size="1.778" layer="95"/>
@@
 </segment>
 <segment>
-<pinref part="U2" gate="G$1" pin="MOSI"/>
+<pinref part="U$2" gate="G$1" pin="MOSI"/>
 <wire x1="-220.98" y1="-83.82" x2="-231.14" y2="-83.82" width="0.1524" layer="91"/>
 <label x="-231.14" y="-83.82" size="1.778" layer="95"/>
@@
 </segment>
 <segment>
-<pinref part="U2" gate="G$1" pin="MISO"/>
+<pinref part="U$2" gate="G$1" pin="MISO"/>
 <wire x1="-220.98" y1="-86.36" x2="-231.14" y2="-86.36" width="0.1524" layer="91"/>
 <label x="-231.14" y="-86.36" size="1.778" layer="95"/>
